Commit message: added robot_base urdf

File: talos_description/urdf/robots/talos.urdf.xacro (robot description, xacro)
@@ -7,16 +7,14 @@
   <!-- The following included files set up definitions of parts of the robot body -->
   <!-- misc common stuff? -->
-  <include filename="$(find talos_description)/urdf/common.xacro" />
-  <!-- youbot base -->
+  <!--include filename="$(find talos_description)/urdf/common.xacro" /-->
+  <!-- talos base -->
   <include filename="$(find talos_description)/urdf/talos_base/base.urdf.xacro" />
-  <!-- youbot arm -->
-  <include filename="$(find talos_description)/urdf/talos_arm/arm.urdf.xacro"/>
-  <!-- youbot gripper -->
-  <include filename="$(find talos_description)/urdf/youbot_gripper/gripper.urdf.xacro" />
+  <!-- talos arm -->
+  <!--include filename="$(find talos_description)/urdf/talos_arm/arm.urdf.xacro"/-->
   <!-- generic simulator_gazebo plugins for starting mechanism control, ros time, ros battery -->
-  <include filename="$(find talos_description)/gazebo/gazebo.urdf.xacro" />
+  <!--include filename="$(find talos_description)/gazebo/gazebo.urdf.xacro" /-->
   <!-- materials for visualization -->
-  <include filename="$(find talos_description)/urdf/materials.urdf.xacro" />
-  <!-- Now we can start using the macros included above to define the actual youbot -->
+  <!--include filename="$(find talos_description)/urdf/materials.urdf.xacro" /-->
+  <!-- Now we can start using the macros included above to define the actual talos -->
   <!-- The first use of a macro.  This one was defined in base.urdf.xacro above.
        A macro like this will expand to a set of link and joint definitions, and to additional
@@ -27,13 +25,7 @@
        is the world frame). For more, see http://www.ros.org/wiki/xacro -->
 <!-- foot for arm-->
-  <xacro:youbot_base name="base"/>
-  <xacro:youbot_plate name="plate" parent="base_link">
-    <origin xyz="-0.159 0 0.046" rpy="0 0 0" />
-  </xacro:youbot_plate>
-  <xacro:youbot_arm name="arm" parent="base_link">
+  <xacro:talos_base name="base"/>
+  <!--xacro:talos_arm name="arm" parent="base_link">
     <origin xyz="0.143 0 0.046" rpy="0 0 0" />
-  </xacro:youbot_arm>
-  <xacro:youbot_gripper name="gripper" parent="arm_link_5">
-    <origin xyz="0 0 0" rpy="0 0 0" />
-  </xacro:youbot_gripper>
+  </xacro:talos_arm-->
 </robot>

File: talos_description/urdf/talos_base/base.gazebo.xacro (robot description, xacro)
@@ -1,5 +1,5 @@
 <?xml version="1.0"?>
 <robot name="talos" xmlns:xacro="http://www.ros.org/wiki/xacro">
-  <xacro:macro name="talos_gazebo">
+  <xacro:macro name="talos_base_gazebo">
     <gazebo>
       <plugin name="object_controller" filename="libgazebo_ros_planar_move.so">
@@ -15,4 +15,25 @@
       <selfCollide>true</selfCollide>
     </gazebo>
+    <!-- front left wheel -->
+    <gazebo reference="wheel_link_fl">
+      <kp>1000000</kp>
+      <kd>100</kd>
+    </gazebo>
+    <gazebo reference="caster_link_fl">
+    </gazebo>
+    <!-- front right wheel -->
+    <gazebo reference="wheel_link_fr">
+      <kp>1000000</kp>
+      <kd>100</kd>
+    </gazebo>
+    <gazebo reference="caster_link_fr">
+    </gazebo>
+    <!-- back left wheel -->
+    <gazebo reference="wheel_link_b">
+      <kp>1000000</kp>
+      <kd>100</kd>
+    </gazebo>
+    <gazebo reference="caster_link_b">
+    </gazebo>
 </xacro:macro>
 </robot>

File: talos_description/urdf/talos_base/base.transmission.xacro (robot description, xacro)
@@ -1,7 +1,7 @@
 <?xml version="1.0"?>
 <robot name="talos" xmlns:xacro="http://www.ros.org/wiki/xacro">
-  <property name="wheel_mechanical_reduction" value="${624/35 * 80/18}"/>
-  <property name="caster_mechanical_reduction" value="${624/35 * 80/18}"/>
-  <property name="" value="0.360"/>
+  <xacro:property name="wheel_mechanical_reduction" value="${624/35 * 80/18}"/>
+  <xacro:property name="caster_mechanical_reduction" value="${624/35 * 80/18}"/>
+  <xacro:property name="w" value="0.360"/>
   <xacro:macro name="talos_base_transmission">
     <!-- front left omni-wheel -->
@@ -10,5 +10,5 @@
       <joint name="wheel_joint_fl"/>
       <actuator name="wheel_motor_fl">
-        <hardwareInterface>EffortJointInterface</hardwareInterface>
+        <hardwareInterface>VelocityJointInterface</hardwareInterface>
         <mechanicalReduction>${wheel_mechanical_reduction}</mechanicalReduction>
       </actuator>
@@ -19,5 +19,5 @@
       <joint name="wheel_joint_fr"/>
       <actuator name="wheel_motor_fr">
-        <hardwareInterface>EffortJointInterface</hardwareInterface>
+        <hardwareInterface>VelocityJointInterface</hardwareInterface>
         <mechanicalReduction>${wheel_mechanical_reduction}</mechanicalReduction>
       </actuator>
@@ -28,5 +28,5 @@
       <joint name="wheel_joint_b"/>
       <actuator name="wheel_motor_b">
-        <hardwareInterface>EffortJointInterface</hardwareInterface>
+        <hardwareInterface>VelocityJointInterface</hardwareInterface>
         <mechanicalReduction>${wheel_mechanical_reduction}</mechanicalReduction>
       </actuator>

File: talos_description/urdf/talos_base/base.urdf.xacro (robot description, xacro)
@@ -2,51 +2,35 @@
 <robot name="talos" xmlns:xacro="http://www.ros.org/wiki/xacro">
   <!-- sensors -->
-  <xacro:include filename="$(find talos_description)/urdf/sensors/sick_tim_561.urdf.xacro"/>
+  <xacro:include filename="$(find talos_description)/urdf/sensors/sick_tim561_laser.urdf.xacro"/>
   <xacro:include filename="$(find talos_description)/urdf/talos_base/base.gazebo.xacro" />
   <xacro:include filename="$(find talos_description)/urdf/talos_base/base.transmission.xacro" />
+  <xacro:property name="M_PI" value="3.141592" />
   <!-- simplified box collision geometry for base -->
-  <property name="base_size_x" value="0.570" />
-  <property name="base_size_y" value="0.360" />
-  <property name="base_size_z" value="0.100" />
-  <property name="base_mass" value="22.0" />
-  <property name="caster_offset_x" value="0.228"  />
-  <property name="caster_offset_y" value="0.158"  />
-  <property name="caster_offset_z" value="-0.034" />
-  <property name="caster_mass" value="0.1" />
-  <property name="wheel_offset_x" value="0.0"  />
-  <property name="wheel_offset_y" value="0.0"  />
-  <property name="wheel_offset_z" value="0.0" />
-  <property name="wheel_mass" value="0.4" />
-  <property name="wheel_radius" value="0.05" />
-  <property name="wheel_length" value="0.005" />
-  <property name="caster_joint_damping" value="1.0" />
-  <property name="caster_joint_friction" value="1.0" />
-  <property name="caster_joint_effort" value="30" />
-  <property name="caster_joint_velocity" value="10" />
-  <property name="caster_joint_safety_k_velocity" value="10.0" />
-  <property name="wheel_joint_damping" value="1.0" />
-  <property name="wheel_joint_friction" value="1.0" />
-  <property name="wheel_joint_effort" value="30" />
-  <property name="wheel_joint_velocity" value="10" />
-  <property name="wheel_joint_safety_k_velocity" value="10.0" />
+  <xacro:property name="base_size_x" value="0.53" />
+  <xacro:property name="base_size_y" value="0.61" />
+  <xacro:property name="base_size_z" value="0.13" />
+  <xacro:property name="base_mass" value="15.0" />
+  <xacro:property name="caster_offset_x" value="0.228"  />
+  <xacro:property name="caster_offset_y" value="0.158"  />
+  <xacro:property name="caster_offset_z" value="-0.034" />
+  <xacro:property name="caster_mass" value="0.1" />
+  <xacro:property name="wheel_offset_x" value="0.0"  />
+  <xacro:property name="wheel_offset_y" value="0.0"  />
+  <xacro:property name="wheel_offset_z" value="0.0" />
+  <xacro:property name="wheel_mass" value="0.4" />
+  <xacro:property name="wheel_radius" value="0.05" />
+  <xacro:property name="wheel_length" value="0.005" />
+  <xacro:property name="caster_joint_damping" value="1.0" />
+  <xacro:property name="caster_joint_friction" value="1.0" />
+  <xacro:property name="caster_joint_effort" value="30" />
+  <xacro:property name="caster_joint_velocity" value="10" />
+  <xacro:property name="caster_joint_safety_k_velocity" value="10.0" />
+  <xacro:property name="wheel_joint_damping" value="1.0" />
+  <xacro:property name="wheel_joint_friction" value="1.0" />
+  <xacro:property name="wheel_joint_effort" value="30" />
+  <xacro:property name="wheel_joint_velocity" value="10" />
+  <xacro:property name="wheel_joint_safety_k_velocity" value="10.0" />
   <xacro:macro name="talos_base" params="name">
     <link name="${name}_footprint">
-      <inertial>
-        <mass value="0.0001" />
-        <origin xyz="0 0 ${-base_size_z / 2.0}" rpy="0 0 0" />
-        <inertia ixx="1.0" ixy="0.0" ixz="0.0" iyy="1.0" iyz="0.0" izz="1.0" />
-      </inertial>
-      <visual>
-        <origin xyz="0 0 0" rpy="0 0 0" />
-        <geometry>
-          <box size="0.001 0.001 0.001" />
-        </geometry>
-      </visual>
-      <collision>
-        <origin xyz="0 0 ${-base_size_z / 2.0}" rpy="0 0 0" />
-        <geometry>
-          <box size="0.001 0.001 0.001" />
-        </geometry>
-      </collision>
     </link>
     <joint name="${name}_footprint_joint" type="fixed">
@@ -64,5 +48,5 @@
         <origin xyz="0 0 0" rpy="0 0 0" />
         <geometry>
-          <mesh filename="package://talos_description/meshes/talos_base/base.dae"/>
+          <mesh filename="package://talos_description/meshes/talos_base/talos_base.stl"/>
         </geometry>
       </visual>
@@ -71,5 +55,5 @@
         <geometry>
           <!--<box size="${base_size_x} ${base_size_y} ${base_size_z}" />-->
-          <mesh filename="package://talos_description/meshes/talos_base/base_convex.dae"/>
+          <mesh filename="package://talos_description/meshes/talos_base/talos_base.stl"/>
         </geometry>
       </collision>
@@ -77,5 +61,5 @@
     <!-- front left omni-wheel -->
     <joint name="caster_joint_fl" type="fixed">
-      <origin xyz="${caster_offset_x} ${caster_offset_y} ${caster_offset_z}" rpy="0 0 0" />
+      <origin xyz="0.118 0.217 0.038" rpy="0 0 -2.0944" />
       <axis xyz="0 0 1" />
       <parent link="${name}_link"/>
@@ -107,5 +91,5 @@
         <origin xyz="0 0 0" rpy="0 0 0" />
         <geometry>
-          <mesh filename="package://talos_description/meshes/talos_base/front-left_wheel.dae" />
+          <mesh filename="package://talos_description/meshes/talos_base/omniwheel.stl" />
         </geometry>
       </visual>
@@ -119,5 +103,5 @@
     <!-- front right omni-wheel -->
     <joint name="caster_joint_fr" type="fixed">
-      <origin xyz="${caster_offset_x} ${-caster_offset_y} ${caster_offset_z}" rpy="0 0 0" />
+      <origin xyz="0.118 -0.211 0.038" rpy="0 ${M_PI} -1.0472" />
       <axis xyz="0 0 1" />
       <parent link="${name}_link"/>
@@ -149,5 +133,5 @@
         <origin xyz="0 0 0" rpy="0 0 0" />
         <geometry>
-          <mesh filename="package://talos_description/meshes/talos_base/front-right_wheel.dae" />
+          <mesh filename="package://talos_description/meshes/talos_base/omniwheel.stl" />
         </geometry>
       </visual>
@@ -161,5 +145,5 @@
     <!-- back omni-wheel -->
     <joint name="caster_joint_b" type="fixed">
-      <origin xyz="${-caster_offset_x} ${caster_offset_y} ${caster_offset_z}" rpy="0 0 0" />
+      <origin xyz="-0.253 0 0.038" rpy="0 0 0" />
       <axis xyz="0 0 1" />
       <parent link="${name}_link"/>
@@ -192,5 +176,5 @@
         <origin xyz="0 0 0" rpy="0 0 0" />
         <geometry>
-          <mesh filename="package://talos_description/meshes/talos_base/back-left_wheel.dae" />
+          <mesh filename="package://talos_description/meshes/talos_base/omniwheel.stl" />
         </geometry>
       </visual>
@@ -203,10 +187,10 @@
     </link>
     <!-- base laser front left-->
-    <xacro:sick_tim561_laser name="${name}_laser_front_left" parent="${name}" ros_topic="scan_front_left" update_rate="15" min_angle="-1.00" max_angle="2.357" >
-      <origin xyz="0.3 0 -0.03" rpy="${M_PI} ${M_PI} ${M_PI}" />
+    <xacro:sick_tim561_laser name="${name}_laser_left" parent="${name}" ros_topic="scan_left" update_rate="15" min_angle="-1.00" max_angle="2.357" >
+      <origin xyz="0.153 0.279 0.07" rpy="0 0 1.0821" />
     </xacro:sick_tim561_laser>
     <!-- base laser front right-->
-    <xacro:sick_tim561_laser name="${name}_laser_front_right" parent="${name}" ros_topic="scan_front_right" update_rate="15" min_angle="-2.357" max_angle="1.00" >
-      <origin xyz="0.3 0 -0.03" rpy="${M_PI} ${M_PI} ${M_PI}" />
+    <xacro:sick_tim561_laser name="${name}_laser_right" parent="${name}" ros_topic="scan_right" update_rate="15" min_angle="-2.357" max_angle="1.00" >
+      <origin xyz="0.153 -0.279 0.07" rpy="0 0 -1.0123" />
     </xacro:sick_tim561_laser>
     <!-- extensions -->
