Commit message: added talos_arm_v1

File: talos_description/urdf/robots/talos.urdf.xacro (robot description, xacro)
@@ -11,5 +11,5 @@
   <include filename="$(find talos_description)/urdf/talos_base/base.urdf.xacro" />
   <!-- talos arm -->
-  <!--include filename="$(find talos_description)/urdf/talos_arm/arm.urdf.xacro"/-->
+  <include filename="$(find talos_description)/urdf/talos_arm/arm.urdf.xacro"/>
   <!-- generic simulator_gazebo plugins for starting mechanism control, ros time, ros battery -->
   <!--include filename="$(find talos_description)/gazebo/gazebo.urdf.xacro" /-->
@@ -26,6 +26,6 @@
 <!-- foot for arm-->
   <xacro:talos_base name="base"/>
-  <!--xacro:talos_arm name="arm" parent="base_link">
-    <origin xyz="0.143 0 0.046" rpy="0 0 0" />
-  </xacro:talos_arm-->
+  <xacro:talos_arm name="arm" parent="base_link">
+    <origin xyz="0.143 0 0.1" rpy="0 0 0" />
+  </xacro:talos_arm>
 </robot>

File: talos_description/urdf/talos_arm/arm.urdf.xacro (robot description, xacro)
@@ -24,5 +24,5 @@
 				<origin xyz="0 0 0" rpy="0 0 0" />
 				<geometry>
-					<mesh filename="package://talos_description/meshes/talos_arm/arm0.dae" />
+					<mesh filename="package://talos_description/meshes/talos_arm/shoulder_link.stl" />
 				</geometry>
 				<material name="DarkGrey" />
@@ -32,5 +32,5 @@
 				<origin xyz="0 0 0" rpy="0 0 0"/>
 				<geometry>
-					<mesh filename="package://talos_description/meshes/talos_arm/arm0_convex.dae" />
+					<mesh filename="package://talos_description/meshes/talos_arm/shoulder_link.stl" />
 					<!--<cylinder length="0.078" radius="0.093"/>-->
 				</geometry>
@@ -39,8 +39,8 @@
 		<!-- joint between arm_0_link and arm_1_link -->
 		<joint name="${name}_joint_1" type="revolute">
-			<origin xyz="0 0 0.05" rpy="0 0 0"/>
+			<origin xyz="0 0 0" rpy="0 0 0"/>
 			<parent link="${name}_link_0"/>
 			<child link="${name}_link_1"/>
-			<axis xyz="0 0 -1"/>
+			<axis xyz="0 1 0"/>
 			<!--<calibration rising="${arm_1_ref}" falling="${arm_1_ref}"/>-->
 			<dynamics damping="1" friction="1" />
@@ -61,7 +61,7 @@
 			</inertial>
 			<visual>
-				<origin xyz="0 0 0" rpy="0 0 0" />
-				<geometry>
-					<mesh filename="package://talos_description/meshes/talos_arm/arm1.dae" />
+				<origin xyz="0.0482 0 0.14" rpy="0 0 0" />
+				<geometry>
+					<mesh filename="package://talos_description/meshes/talos_arm/biceps_link.stl" />
 				</geometry>
 				<!--<material name="Orange" />-->
@@ -69,7 +69,7 @@
 			<collision>
 				<!--<origin xyz="0 0 -0.003" rpy="0 0 0" />-->
-				<origin xyz="0 0 0" rpy="0 0 0" />
-				<geometry>
-					<mesh filename="package://talos_description/meshes/talos_arm/arm1_convex.dae" />
+				<origin xyz="0.0482 0 0.14" rpy="0 0 0" />
+				<geometry>
+					<mesh filename="package://talos_description/meshes/talos_arm/biceps_link.stl" />
 					<!--<cylinder length="0.102" radius="0.080"/>-->
 				</geometry>
@@ -78,5 +78,5 @@
 		<!-- joint between arm_1_link and arm_2_link -->
 		<joint name="${name}_joint_2" type="revolute">
-			<origin xyz="0.033 0 0.019" rpy="0 ${-65 * M_PI / 180} 0"/>
+			<origin xyz="0.0482 0 0.142" rpy="0 ${M_PI / 2} 0"/>
 			<parent link="${name}_link_1"/>
 			<child link="${name}_link_2"/>
@@ -93,15 +93,15 @@
 			</inertial>
 			<visual>
-			<origin xyz="0 -0.032 0.078" rpy="0 0 0" />
-				<geometry>
-					<mesh filename="package://talos_description/meshes/talos_arm/arm2.dae" />
-				</geometry>
-				<material name="Orange" />
+			<origin xyz="0 0 0.142" rpy="0 0 0" />
+				<geometry>
+					<mesh filename="package://talos_description/meshes/talos_arm/forearm_link.stl" />
+				</geometry>
+				<material name="Black" />
 			</visual>
 			<collision>
 				<!--<origin xyz="0.001 -0.041 0.074" rpy="0 0 0" />-->
-				<origin xyz="0 -0.032 0.078" rpy="0 0 0" />
-				<geometry>
-					<mesh filename="package://talos_description/meshes/talos_arm/arm2_convex.dae" />
+				<origin xyz="0 0 0.142" rpy="0 0 0" />
+				<geometry>
+					<mesh filename="package://talos_description/meshes/talos_arm/forearm_link.stl" />
 					<!--<box size="0.074 0.082 0.222"/>-->
 				</geometry>
@@ -109,6 +109,6 @@
 		</link>
 		<!-- joint between arm_2_link and arm_3_link -->
-		<!--<joint name="${name}_joint_3" type="revolute">
-			<origin xyz="0.000 0.000 0.155" rpy="0 ${146 * M_PI / 180} 0"/>
+		<joint name="${name}_joint_3" type="revolute">
+			<origin xyz="0 0 0.142" rpy="0 0 0"/>
 			<parent link="${name}_link_2"/>
 			<child link="${name}_link_3"/>
@@ -116,13 +116,4 @@
 			<dynamics damping="1" friction="1" />
 			<limit effort="${6}" velocity="${M_PI / 2.0}" lower="-${joint_3_limit}" upper="0"/>
-                        <safety_controller k_position="20" k_velocity="50" soft_lower_limit="-${joint_3_limit_soft}" soft_upper_limit="${threshold}" />
-		</joint>-->
-		<joint name="${name}_joint_3" type="revolute">
-			<origin xyz="0.000 0.000 0.155" rpy="0 ${146 * M_PI / 180} 0"/>
-			<parent link="${name}_link_2"/>
-			<child link="${name}_link_3"/>
-			<axis xyz="0 1 0"/>
-			<dynamics damping="1" friction="1" />
-			<limit effort="${6}" velocity="${M_PI / 2.0}" lower="-${joint_3_limit}" upper="0"/>
                         <safety_controller k_position="20" k_velocity="50" soft_lower_limit="-${joint_3_limit_soft}" soft_upper_limit="-${threshold}" />
 		</joint>
@@ -133,7 +124,7 @@
 			</inertial>
 			<visual>
-				<origin xyz="0.000 0.028 0.079" rpy="0 0 0" />
-				<geometry>
-					<mesh filename="package://talos_description/meshes/talos_arm/arm3.dae" />
+				<origin xyz="0 0 0" rpy="0 0 0" />
+				<geometry>
+					<mesh filename="package://talos_description/meshes/talos_arm/wrist_1_link.stl" />
 				</geometry>
 				<material name="Orange" />
@@ -141,7 +132,7 @@
 			<collision>
 				<!--<origin xyz="0.000 0.025 0.067" rpy="0 0 0" />-->
-				<origin xyz="0.000 0.028 0.079" rpy="0 0 0" />
-				<geometry>
-					<mesh filename="package://talos_description/meshes/talos_arm/arm3_convex.dae" />
+				<origin xyz="0 0 0" rpy="0 0 0" />
+				<geometry>
+					<mesh filename="package://talos_description/meshes/talos_arm/wrist_1_link.stl" />
 					<!--<box size="0.064 0.054 0.192"/>-->
 				</geometry>
@@ -150,8 +141,8 @@
 		<!-- joint between arm_3_link and arm_4_link -->
 		<joint name="${name}_joint_4" type="revolute">
-			<origin xyz="0.000 0.000 0.135" rpy="0 ${-102.5 * M_PI / 180} 0" />
+			<origin xyz="0 0 0.0715" rpy="0 0 0" />
 			<parent link="${name}_link_3"/>
 			<child link="${name}_link_4"/>
-			<axis xyz="0 1 0" />
+			<axis xyz="0 0 1" />
 			<!--<calibration rising="${arm_4_ref}" falling="${arm_4_ref}"/>-->
 			<dynamics damping="1" friction="1" />
@@ -165,7 +156,7 @@
 			</inertial>
 			<visual>
-				<origin xyz="0 -0.010 0.029" rpy="0 0 0"/>
-				<geometry>
-					<mesh filename="package://talos_description/meshes/talos_arm/arm4.dae" />
+				<origin xyz="0 0 0.043" rpy="0 0 0"/>
+				<geometry>
+					<mesh filename="package://talos_description/meshes/talos_arm/wrist_2_link.stl" />
 				</geometry>
 				<material name="Orange" />
@@ -173,7 +164,7 @@
 			<collision>
 				<!--<origin xyz="0 0 0.026" rpy="0 0 0" />-->
-				<origin xyz="0 -0.010 0.029" rpy="0 0 0"/>
-				<geometry>
-					<mesh filename="package://talos_description/meshes/talos_arm/arm4_convex.dae" />
+				<origin xyz="0 0 0.043" rpy="0 0 0"/>
+				<geometry>
+					<mesh filename="package://talos_description/meshes/talos_arm/wrist_2_link.stl" />
 					<!--<box size="0.058 0.100 0.118"/>-->
 				</geometry>
@@ -181,9 +172,41 @@
 		</link>
 		<!-- joint between arm_4_link and arm_5_link -->
-		<joint name="${name}_joint_5" type="revolute">
-			<origin xyz="-0.002 0 0.130" rpy="0 0 ${167.5 * M_PI / 180}" />
+		<joint name="${name}_joint_5" type="fixed">
+			<origin xyz="0 0 0.043" rpy="0 0 0" />
 			<parent link="${name}_link_4"/>
 			<child link="${name}_link_5"/>
-			<axis xyz="0 0 -1" />
+			<axis xyz="0 0 1" />
+			<!--<calibration rising="${arm_4_ref}" falling="${arm_4_ref}"/>-->
+			<dynamics damping="1" friction="1" />
+			<limit effort="${2}" velocity="${M_PI / 2.0}" lower="0" upper="${joint_4_limit}"/>
+			<safety_controller k_position="20" k_velocity="100" soft_lower_limit="0" soft_upper_limit="${joint_4_limit_soft}" />
+		</joint>
+		<link name="${name}_link_5">
+			<inertial>
+				<mass value="${link_5_mass}"/>
+				<xacro:link_4_inertia_tensor />
+			</inertial>
+			<visual>
+				<origin xyz="0 0 0" rpy="0 0 1.57"/>
+				<geometry>
+					<mesh filename="package://talos_description/meshes/talos_arm/gripper_rail_link.stl" />
+				</geometry>
+				<material name="Orange" />
+			</visual>
+			<collision>
+				<!--<origin xyz="0 0 0.026" rpy="0 0 0" />-->
+				<origin xyz="0 0 0" rpy="0 0 1.57"/>
+				<geometry>
+					<mesh filename="package://talos_description/meshes/talos_arm/gripper_rail_link.stl" />
+					<!--<box size="0.058 0.100 0.118"/>-->
+				</geometry>
+			</collision>
+		</link>
+		<!-- joint between arm_5_link and arm_6_link -->
+		<joint name="${name}_joint_6" type="prismatic">
+			<origin xyz="0 0 0" rpy="0 0 0" />
+			<parent link="${name}_link_5"/>
+			<child link="${name}_link_6"/>
+			<axis xyz="0 -1 0" />
 			<!--<calibration rising="${arm_5_ref}" falling="${arm_5_ref}"/>-->
 			<dynamics damping="1" friction="1" />
@@ -191,20 +214,51 @@
                         <safety_controller k_position="20" k_velocity="100" soft_lower_limit="0" soft_upper_limit="${joint_5_limit_soft}" />
 		</joint>
-		<link name="${name}_link_5">
-			<inertial>
-				<mass value="${link_5_mass}"/>
-				<xacro:link_5_inertia_tensor />
-			</inertial>
-			<visual>
-				<origin xyz="0.003 0 -0.034" rpy="0 0 0" />
-				<geometry>
-					<mesh filename="package://talos_description/meshes/talos_arm/arm5.dae" />
+		<link name="${name}_link_6">
+			<inertial>
+				<mass value="${link_6_mass}"/>
+				<xacro:link_6_inertia_tensor />
+			</inertial>
+			<visual>
+				<origin xyz="0 0 0" rpy="0 0 1.57" />
+				<geometry>
+					<mesh filename="package://talos_description/meshes/talos_arm/gripper_hand_fixed_link.stl" />
 				</geometry>
 				<material name="DarkGrey" />
 			</visual>
 			<collision>
-				<origin xyz="0.003 0 -0.034" rpy="0 0 0" />
-				<geometry>
-					<mesh filename="package://talos_description/meshes/talos_arm/arm5_convex.dae" />
+				<origin xyz="0 0 0" rpy="0 0 1.57" />
+				<geometry>
+					<mesh filename="package://talos_description/meshes/talos_arm/gripper_hand_fixed_link.stl" />
+					<!--<box size="0.054 0.096 0.030"/>-->
+				</geometry>
+			</collision>
+		</link>
+		<!-- joint between arm_5_link and arm_7_link -->
+		<joint name="${name}_joint_7" type="revolute">
+			<origin xyz="0 0 0" rpy="0 0 0" />
+			<parent link="${name}_link_5"/>
+			<child link="${name}_link_7"/>
+			<axis xyz="0 1 0" />
+			<!--<calibration rising="${arm_5_ref}" falling="${arm_5_ref}"/>-->
+			<dynamics damping="1" friction="1" />
+			<limit effort="1" velocity="${M_PI / 2.0}" lower="0" upper="${joint_5_limit}" />
+                        <safety_controller k_position="20" k_velocity="100" soft_lower_limit="0" soft_upper_limit="${joint_5_limit_soft}" />
+		</joint>
+		<link name="${name}_link_7">
+			<inertial>
+				<mass value="${link_7_mass}"/>
+				<xacro:link_7_inertia_tensor />
+			</inertial>
+			<visual>
+				<origin xyz="0 0 0" rpy="0 0 -1.57" />
+				<geometry>
+					<mesh filename="package://talos_description/meshes/talos_arm/gripper_hand_fixed_link.stl" />
+				</geometry>
+				<material name="DarkGrey" />
+			</visual>
+			<collision>
+				<origin xyz="0 0 0" rpy="0 0 -1.57" />
+				<geometry>
+					<mesh filename="package://talos_description/meshes/talos_arm/gripper_hand_fixed_link.stl" />
 					<!--<box size="0.054 0.096 0.030"/>-->
 				</geometry>

Commit message: modified base_arm

File: talos_description/urdf/robots/talos.urdf.xacro (robot description, xacro)
@@ -27,5 +27,5 @@
   <xacro:talos_base name="base"/>
   <xacro:talos_arm name="arm" parent="base_link">
-    <origin xyz="0.143 0 0.1" rpy="0 0 0" />
+    <origin xyz="0.147 0 0.147" rpy="0 0 0" />
   </xacro:talos_arm>
 </robot>

Commit message: added urdf

File: talos_description/urdf/robots/talos.urdf.xacro (robot description, xacro)
@@ -25,5 +25,5 @@
        is the world frame). For more, see http://www.ros.org/wiki/xacro -->
 <!-- foot for arm-->
-  <xacro:talos_base name="base"/>
+  <xacro:macro name = "talos_base" params ="base"/>
   <!--xacro:talos_arm name="arm" parent="base_link">
     <origin xyz="0.143 0 0.046" rpy="0 0 0" />

File: talos_description/urdf/sensors/sick_tim561_laser.urdf.xacro (robot description, xacro)
@@ -2,5 +2,5 @@
 <robot name="talos" xmlns:xacro="http://ros.org/wiki/xacro">
   <xacro:include filename="$(find talos_description)/urdf/sensors/sick_tim561_laser.gazebo.xacro" />
-  <xacro:macro name="sick_tim561_laser" params="name parent *origin ros_topic update_rate min_angle max_angle">
+  <xacro:macro name="sick_tim561_laser" params="laser parent *origin ros_topic update_rate min_angle max_angle">
     <joint name="${name}_sick_tim561_laser_joint" type="fixed">
       <axis xyz="0 1 0" />
@@ -30,5 +30,5 @@
  </link>
  <!-- gazebo extensions -->
- <xacro:sick_tim561_laser_gazebo name="${name}" ros_topic="${ros_topic}" update_rate="${update_rate}" min_angle="${min_angle}" max_angle="${max_angle}" />
+ <xacro:sick_tim561_laser_gazebo laser_name="${name}" ros_topic="${ros_topic}" update_rate="${update_rate}" min_angle="${min_angle}" max_angle="${max_angle}" />
 </xacro:macro>
 </robot>

File: talos_description/urdf/talos_base/base.urdf.xacro (robot description, xacro)
@@ -7,11 +7,5 @@
   <xacro:property name="M_PI" value="3.141592" />
   <!-- simplified box collision geometry for base -->
-  <xacro:property name="base_size_x" value="0.53" />
-  <xacro:property name="base_size_y" value="0.61" />
-  <xacro:property name="base_size_z" value="0.13" />
   <xacro:property name="base_mass" value="15.0" />
-  <xacro:property name="caster_offset_x" value="0.228"  />
-  <xacro:property name="caster_offset_y" value="0.158"  />
-  <xacro:property name="caster_offset_z" value="-0.034" />
   <xacro:property name="caster_mass" value="0.1" />
   <xacro:property name="wheel_offset_x" value="0.0"  />
@@ -20,10 +14,4 @@
   <xacro:property name="wheel_mass" value="0.4" />
   <xacro:property name="wheel_radius" value="0.05" />
-  <xacro:property name="wheel_length" value="0.005" />
-  <xacro:property name="caster_joint_damping" value="1.0" />
-  <xacro:property name="caster_joint_friction" value="1.0" />
-  <xacro:property name="caster_joint_effort" value="30" />
-  <xacro:property name="caster_joint_velocity" value="10" />
-  <xacro:property name="caster_joint_safety_k_velocity" value="10.0" />
   <xacro:property name="wheel_joint_damping" value="1.0" />
   <xacro:property name="wheel_joint_friction" value="1.0" />
