Commit message: fixed xacro-noetic issues

File: talos_description/urdf/robots/talos.urdf.xacro (robot description, xacro)
@@ -9,5 +9,5 @@
   <!--include filename="$(find talos_description)/urdf/common.xacro" /-->
   <!-- talos base -->
-  <include filename="$(find talos_description)/urdf/talos_base/base.urdf.xacro" />
+  <xacro:include filename="$(find talos_description)/urdf/talos_base/base.urdf.xacro" />
   <!-- talos arm -->
   <!--include filename="$(find talos_description)/urdf/talos_arm/arm.urdf.xacro"/-->
@@ -15,5 +15,5 @@
   <!--include filename="$(find talos_description)/gazebo/gazebo.urdf.xacro" /-->
   <!-- materials for visualization -->
-  <!--include filename="$(find talos_description)/urdf/materials.urdf.xacro" /-->
+  <include filename="$(find talos_description)/urdf/materials.urdf.xacro" />
   <!-- Now we can start using the macros included above to define the actual talos -->
   <!-- The first use of a macro.  This one was defined in base.urdf.xacro above.
@@ -25,5 +25,5 @@
        is the world frame). For more, see http://www.ros.org/wiki/xacro -->
 <!-- foot for arm-->
-  <xacro:macro name = "talos_base" params ="base"/>
+  <xacro:talos_base name ="base"/>
   <!--xacro:talos_arm name="arm" parent="base_link">
     <origin xyz="0.143 0 0.046" rpy="0 0 0" />

File: talos_description/urdf/sensors/sick_tim561_laser.gazebo.xacro (robot description, xacro)
@@ -27,7 +27,6 @@
                     <alwaysOn>true</alwaysOn>
                     <updateRate>${update_rate}</updateRate>
-                    <topicName>${ros_topic}</topicName>
+                    <topicName>/${ros_topic}</topicName>
                     <frameName>${name}_link</frameName>
-                    <interface:laser name="gazebo_ros_${name}_iface" />
                 </plugin>
             </sensor>

File: talos_description/urdf/sensors/sick_tim561_laser.urdf.xacro (robot description, xacro)
@@ -2,8 +2,8 @@
 <robot name="talos" xmlns:xacro="http://ros.org/wiki/xacro">
   <xacro:include filename="$(find talos_description)/urdf/sensors/sick_tim561_laser.gazebo.xacro" />
-  <xacro:macro name="sick_tim561_laser" params="laser parent *origin ros_topic update_rate min_angle max_angle">
+  <xacro:macro name="sick_tim561_laser" params="name parent *origin ros_topic update_rate min_angle max_angle">
     <joint name="${name}_sick_tim561_laser_joint" type="fixed">
       <axis xyz="0 1 0" />
-      <insert_block name="origin" />
+      <xacro:insert_block name="origin" />
       <parent link="${parent}_link"/>
       <child link="${name}_link"/>
@@ -12,16 +12,15 @@
       <inertial>
         <mass value="0.16" />
-        <origin xyz="0 0 0" rpy="0 0 0" />
+        <origin xyz="0 0 0.04" rpy="0 0 0" />
         <inertia ixx="0.1" ixy="0" ixz="0" iyy="0.1" iyz="0" izz="0.1" />
       </inertial>
       <visual>
-      	<origin xyz="0 0 0" rpy="0 0 0" />
+      	<origin xyz="0 0 0.04" rpy="0 0 0" />
        <geometry>
         <mesh filename="package://talos_description/meshes/sensors/sick_tim561.stl" />
       </geometry>
-      <material name="DarkGrey" />
     </visual>
     <collision>
-      <origin xyz="0 0 0" rpy="0 0 0" />
+      <origin xyz="0 0 0.04" rpy="0 0 0" />
       <geometry>
        <mesh filename="package://talos_description/meshes/sensors/sick_tim561.stl" />
@@ -30,5 +29,5 @@
  </link>
  <!-- gazebo extensions -->
- <xacro:sick_tim561_laser_gazebo laser_name="${name}" ros_topic="${ros_topic}" update_rate="${update_rate}" min_angle="${min_angle}" max_angle="${max_angle}" />
+ <xacro:sick_tim561_laser_gazebo name="${name}" ros_topic="${ros_topic}" update_rate="${update_rate}" min_angle="${min_angle}" max_angle="${max_angle}" />
 </xacro:macro>
 </robot>

File: talos_description/urdf/talos_arm/arm.urdf.xacro (robot description, xacro)
@@ -6,5 +6,5 @@
 	<include filename="$(find talos_description)/urdf/talos_arm/arm.gazebo.xacro" />
 	<include filename="$(find talos_description)/urdf/talos_arm/arm.transmission.xacro" />
-        <include filename="$(find talos_description)/urdf/talos_arm/limits.urdf.xacro" />
+    <include filename="$(find talos_description)/urdf/talos_arm/limits.urdf.xacro" />
 	<xacro:macro name="talos_arm" params="parent name *origin">
 		<!-- joint between base_link and arm_0_link -->

File: talos_description/urdf/talos_base/base.gazebo.xacro (robot description, xacro)
@@ -1,9 +1,12 @@
 <?xml version="1.0"?>
-<robot name="talos" xmlns:xacro="http://www.ros.org/wiki/xacro">
+<robot  xmlns:sensor="http://playerstage.sourceforge.net/gazebo/xmlschema/#sensor"
+        xmlns:controller="http://playerstage.sourceforge.net/gazebo/xmlschema/#controller"
+        xmlns:interface="http://playerstage.sourceforge.net/gazebo/xmlschema/#interface"
+        xmlns:xacro="http://ros.org/wiki/xacro">
   <xacro:macro name="talos_base_gazebo">
     <gazebo>
       <plugin name="object_controller" filename="libgazebo_ros_planar_move.so">
-        <commandTopic>cmd_vel</commandTopic>
-        <odometryTopic>odom</odometryTopic>
+        <commandTopic>/cmd_vel</commandTopic>
+        <odometryTopic>/odom</odometryTopic>
         <odometryFrame>odom</odometryFrame>
         <odometryRate>20.0</odometryRate>
@@ -11,5 +14,6 @@
       </plugin>
     </gazebo>
-    <gazebo reference="${name}_footprint">
+  </xacro:macro>
+    <gazebo reference="talos_base">
       <gravity>true</gravity>
       <selfCollide>true</selfCollide>
@@ -17,6 +21,12 @@
     <!-- front left wheel -->
     <gazebo reference="wheel_link_fl">
-      <kp>1000000</kp>
-      <kd>100</kd>
+      <dampingFactor>100000</dampingFactor>
+      <kp>100000.0</kp>
+      <kd>1000.0</kd>
+      <mu1>0</mu1>
+      <mu2>0</mu2>
+      <fdir>1 0 0</fdir>
+      <maxVel>1.0</maxVel>
+      <minDepth>0.0</minDepth>
     </gazebo>
     <gazebo reference="caster_link_fl">
@@ -24,6 +34,12 @@
     <!-- front right wheel -->
     <gazebo reference="wheel_link_fr">
-      <kp>1000000</kp>
-      <kd>100</kd>
+      <dampingFactor>100000</dampingFactor>
+      <kp>100000.0</kp>
+      <kd>1000.0</kd>
+      <mu1>0</mu1>
+      <mu2>0</mu2>
+      <fdir>1 0 0</fdir>
+      <maxVel>1.0</maxVel>
+      <minDepth>0.0</minDepth>
     </gazebo>
     <gazebo reference="caster_link_fr">
@@ -31,9 +47,14 @@
     <!-- back left wheel -->
     <gazebo reference="wheel_link_b">
-      <kp>1000000</kp>
-      <kd>100</kd>
+      <dampingFactor>100000</dampingFactor>
+      <kp>100000.0</kp>
+      <kd>1000.0</kd>
+      <mu1>0</mu1>
+      <mu2>0</mu2>
+      <fdir>1 0 0</fdir>
+      <maxVel>1.0</maxVel>
+      <minDepth>0.0</minDepth>
     </gazebo>
     <gazebo reference="caster_link_b">
     </gazebo>
-</xacro:macro>
 </robot>

File: talos_description/urdf/talos_base/base.transmission.xacro (robot description, xacro)
@@ -1,4 +1,7 @@
 <?xml version="1.0"?>
-<robot name="talos" xmlns:xacro="http://www.ros.org/wiki/xacro">
+<robot  xmlns:sensor="http://playerstage.sourceforge.net/gazebo/xmlschema/#sensor"
+        xmlns:controller="http://playerstage.sourceforge.net/gazebo/xmlschema/#controller"
+        xmlns:interface="http://playerstage.sourceforge.net/gazebo/xmlschema/#interface"
+        xmlns:xacro="http://ros.org/wiki/xacro">
   <xacro:property name="wheel_mechanical_reduction" value="${624/35 * 80/18}"/>
   <xacro:property name="caster_mechanical_reduction" value="${624/35 * 80/18}"/>

File: talos_description/urdf/talos_base/base.urdf.xacro (robot description, xacro)
@@ -1,4 +1,7 @@
 <?xml version="1.0"?>
-<robot name="talos" xmlns:xacro="http://www.ros.org/wiki/xacro">
+<robot  xmlns:sensor="http://playerstage.sourceforge.net/gazebo/xmlschema/#sensor"
+        xmlns:controller="http://playerstage.sourceforge.net/gazebo/xmlschema/#controller"
+        xmlns:interface="http://playerstage.sourceforge.net/gazebo/xmlschema/#interface"
+        xmlns:xacro="http://ros.org/wiki/xacro">
   <!-- sensors -->
   <xacro:include filename="$(find talos_description)/urdf/sensors/sick_tim561_laser.urdf.xacro"/>
@@ -19,7 +22,6 @@
   <xacro:property name="wheel_joint_velocity" value="10" />
   <xacro:property name="wheel_joint_safety_k_velocity" value="10.0" />
-  <xacro:macro name="talos_base" params="name">
-    <link name="${name}_footprint">
-    </link>
+  <xacro:macro name = "talos_base" params="name">
+    <link name="${name}_footprint"/>
     <joint name="${name}_footprint_joint" type="fixed">
       <origin xyz="0 0 0" rpy="0 0 0" />
@@ -175,10 +177,10 @@
     </link>
     <!-- base laser front left-->
-    <xacro:sick_tim561_laser name="${name}_laser_left" parent="${name}" ros_topic="scan_left" update_rate="15" min_angle="-1.00" max_angle="2.357" >
-      <origin xyz="0.153 0.279 0.07" rpy="0 0 1.0821" />
+    <xacro:sick_tim561_laser name="${name}_laser_left" parent="${name}" ros_topic="scan_left" update_rate="15" min_angle="-2.2" max_angle="2.5" >
+      <origin xyz="0.153 0.279 0.03" rpy="0 0 1.0821" />
     </xacro:sick_tim561_laser>
     <!-- base laser front right-->
-    <xacro:sick_tim561_laser name="${name}_laser_right" parent="${name}" ros_topic="scan_right" update_rate="15" min_angle="-2.357" max_angle="1.00" >
-      <origin xyz="0.153 -0.279 0.07" rpy="0 0 -1.0123" />
+    <xacro:sick_tim561_laser name="${name}_laser_right" parent="${name}" ros_topic="scan_right" update_rate="15" min_angle="-2.5" max_angle="2.2" >
+      <origin xyz="0.153 -0.27 0.03" rpy="0 0 -1.0821" />
     </xacro:sick_tim561_laser>
     <!-- extensions -->
