Commit message: armv0 updated

File: talos_description/urdf/robots/talos.urdf.xacro (robot description, xacro)
@@ -11,5 +11,5 @@
   <xacro:include filename="$(find talos_description)/urdf/talos_base/base.urdf.xacro" />
   <!-- talos arm -->
-  <!--include filename="$(find talos_description)/urdf/talos_arm/arm.urdf.xacro"/-->
+  <xacro:include filename="$(find talos_description)/urdf/talos_arm/arm.urdf.xacro"/>
   <!-- generic simulator_gazebo plugins for starting mechanism control, ros time, ros battery -->
   <!--include filename="$(find talos_description)/gazebo/gazebo.urdf.xacro" /-->
@@ -26,6 +26,6 @@
 <!-- foot for arm-->
   <xacro:talos_base name ="base"/>
-  <!--xacro:talos_arm name="arm" parent="base_link">
-    <origin xyz="0.143 0 0.046" rpy="0 0 0" />
-  </xacro:talos_arm-->
+  <xacro:talos_arm name="arm" parent="base_link">
+    <origin xyz="0.143 0 0.147" rpy="0 0 0" />
+  </xacro:talos_arm>
 </robot>

File: talos_description/urdf/talos_arm/arm.urdf.xacro (robot description, xacro)
@@ -4,11 +4,15 @@
         xmlns:interface="http://playerstage.sourceforge.net/gazebo/xmlschema/#interface"
         xmlns:xacro="http://ros.org/wiki/xacro">
-	<include filename="$(find talos_description)/urdf/talos_arm/arm.gazebo.xacro" />
-	<include filename="$(find talos_description)/urdf/talos_arm/arm.transmission.xacro" />
-    <include filename="$(find talos_description)/urdf/talos_arm/limits.urdf.xacro" />
+	<xacro:include filename="$(find talos_description)/urdf/talos_arm/arm.gazebo.xacro" />
+	<xacro:include filename="$(find talos_description)/urdf/talos_arm/arm.transmission.xacro" />
+    <xacro:include filename="$(find talos_description)/urdf/talos_arm/limits.urdf.xacro" />
+	<xacro:include filename="$(find realsense2_description)/urdf/_d435.urdf.xacro"/>
 	<xacro:macro name="talos_arm" params="parent name *origin">
+		<xacro:sensor_d435 name="camera" topics_ns="camera" parent="${name}_link_4" publish_pointcloud="true">
+			<origin xyz="0.025 0.0 0.01" rpy="0 0 0" />
+		</xacro:sensor_d435>
 		<!-- joint between base_link and arm_0_link -->
 		<joint name="${name}_joint_0" type="fixed" >
-			<insert_block name="origin" />
+			<xacro:insert_block name="origin" />
 			<parent link="${parent}" />
 			<child link="${name}_link_0" />
@@ -24,7 +28,7 @@
 				<origin xyz="0 0 0" rpy="0 0 0" />
 				<geometry>
-					<mesh filename="package://talos_description/meshes/talos_arm/arm0.dae" />
-				</geometry>
-				<material name="DarkGrey" />
+					<mesh filename="package://talos_description/meshes/talos_arm/shoulder_link.stl" />
+				</geometry>
+				<!--material name="DarkGrey" /-->
 			</visual>
 			<collision>
@@ -32,5 +36,5 @@
 				<origin xyz="0 0 0" rpy="0 0 0"/>
 				<geometry>
-					<mesh filename="package://talos_description/meshes/talos_arm/arm0_convex.dae" />
+					<mesh filename="package://talos_description/meshes/talos_arm/shoulder_link.stl" />
 					<!--<cylinder length="0.078" radius="0.093"/>-->
 				</geometry>
@@ -39,16 +43,15 @@
 		<!-- joint between arm_0_link and arm_1_link -->
 		<joint name="${name}_joint_1" type="revolute">
-			<origin xyz="0 0 0.05" rpy="0 0 0"/>
+			<origin xyz="0 0 0" rpy="0 0 0"/>
 			<parent link="${name}_link_0"/>
 			<child link="${name}_link_1"/>
-			<axis xyz="0 0 -1"/>
+			<axis xyz="0 1 0"/>
 			<!--<calibration rising="${arm_1_ref}" falling="${arm_1_ref}"/>-->
-			<dynamics damping="1" friction="1" />
+			<dynamics damping="10" friction="10" />
 			<!-- damping - N*s/m, N*s*m/rad -->
 			<!-- friction - N, N*m -->
-			<limit effort="${9.5}" velocity="${M_PI / 2.0}" lower="0" upper="${joint_1_limit}"/>
+			<limit effort="100" velocity="${M_PI / 2.0}" lower="-${joint_1_limit}" upper="${joint_1_limit}"/>
 			<!--effort - N, N*m-->
 			<!--velocity - m/s, rad/s-->
-			<safety_controller k_position="20" k_velocity="${9.5/M_PI / 2.0}" soft_lower_limit="${threshold}" soft_upper_limit="${joint_1_limit_soft}" />
 			<!--k_position N/m, N/rad-->
 			<!--k_velocity N*s/m, N*s*m/rad-->
@@ -61,7 +64,7 @@
 			</inertial>
 			<visual>
-				<origin xyz="0 0 0" rpy="0 0 0" />
-				<geometry>
-					<mesh filename="package://talos_description/meshes/talos_arm/arm1.dae" />
+				<origin xyz="0.0482 0 0.14" rpy="0 0 0" />
+				<geometry>
+					<mesh filename="package://talos_description/meshes/talos_arm/biceps_link.stl" />
 				</geometry>
 				<!--<material name="Orange" />-->
@@ -69,7 +72,7 @@
 			<collision>
 				<!--<origin xyz="0 0 -0.003" rpy="0 0 0" />-->
-				<origin xyz="0 0 0" rpy="0 0 0" />
-				<geometry>
-					<mesh filename="package://talos_description/meshes/talos_arm/arm1_convex.dae" />
+				<origin xyz="0.0482 0 0.14" rpy="0 0 0" />
+				<geometry>
+					<mesh filename="package://talos_description/meshes/talos_arm/biceps_link.stl" />
 					<!--<cylinder length="0.102" radius="0.080"/>-->
 				</geometry>
@@ -78,12 +81,11 @@
 		<!-- joint between arm_1_link and arm_2_link -->
 		<joint name="${name}_joint_2" type="revolute">
-			<origin xyz="0.033 0 0.019" rpy="0 ${-65 * M_PI / 180} 0"/>
+			<origin xyz="0.0482 0 0.142" rpy="0 ${M_PI / 2} 0"/>
 			<parent link="${name}_link_1"/>
 			<child link="${name}_link_2"/>
 			<axis xyz="0 1 0"/>
 			<!--<calibration rising="${arm_2_ref}" falling="${arm_2_ref}"/>-->
-			<dynamics damping="1" friction="1" />
-			<limit effort="${9.5}" velocity="${M_PI / 2.0}" lower="0" upper="${joint_2_limit}"/>
-                        <safety_controller k_position="20" k_velocity="${2*9.5/M_PI}" soft_lower_limit="${threshold}" soft_upper_limit="${joint_2_limit_soft}" />
+			<dynamics damping="10" friction="10" />
+			<limit effort="100" velocity="${M_PI / 2.0}" lower="-${joint_2_limit}" upper="${joint_2_limit}"/>
 		</joint>
 		<link name="${name}_link_2">
@@ -93,15 +95,15 @@
 			</inertial>
 			<visual>
-			<origin xyz="0 -0.032 0.078" rpy="0 0 0" />
-				<geometry>
-					<mesh filename="package://talos_description/meshes/talos_arm/arm2.dae" />
-				</geometry>
-				<material name="Orange" />
+			<origin xyz="0 0 0.142" rpy="0 0 0" />
+				<geometry>
+					<mesh filename="package://talos_description/meshes/talos_arm/forearm_link.stl" />
+				</geometry>
+				<!--material name="Black" /-->
 			</visual>
 			<collision>
 				<!--<origin xyz="0.001 -0.041 0.074" rpy="0 0 0" />-->
-				<origin xyz="0 -0.032 0.078" rpy="0 0 0" />
-				<geometry>
-					<mesh filename="package://talos_description/meshes/talos_arm/arm2_convex.dae" />
+				<origin xyz="0 0 0.142" rpy="0 0 0" />
+				<geometry>
+					<mesh filename="package://talos_description/meshes/talos_arm/forearm_link.stl" />
 					<!--<box size="0.074 0.082 0.222"/>-->
 				</geometry>
@@ -109,21 +111,11 @@
 		</link>
 		<!-- joint between arm_2_link and arm_3_link -->
-		<!--<joint name="${name}_joint_3" type="revolute">
-			<origin xyz="0.000 0.000 0.155" rpy="0 ${146 * M_PI / 180} 0"/>
+		<joint name="${name}_joint_3" type="revolute">
+			<origin xyz="0 0 0.142" rpy="0 0 0"/>
 			<parent link="${name}_link_2"/>
 			<child link="${name}_link_3"/>
 			<axis xyz="0 1 0"/>
-			<dynamics damping="1" friction="1" />
-			<limit effort="${6}" velocity="${M_PI / 2.0}" lower="-${joint_3_limit}" upper="0"/>
-                        <safety_controller k_position="20" k_velocity="50" soft_lower_limit="-${joint_3_limit_soft}" soft_upper_limit="${threshold}" />
-		</joint>-->
-		<joint name="${name}_joint_3" type="revolute">
-			<origin xyz="0.000 0.000 0.155" rpy="0 ${146 * M_PI / 180} 0"/>
-			<parent link="${name}_link_2"/>
-			<child link="${name}_link_3"/>
-			<axis xyz="0 1 0"/>
-			<dynamics damping="1" friction="1" />
-			<limit effort="${6}" velocity="${M_PI / 2.0}" lower="-${joint_3_limit}" upper="0"/>
-                        <safety_controller k_position="20" k_velocity="50" soft_lower_limit="-${joint_3_limit_soft}" soft_upper_limit="-${threshold}" />
+			<dynamics damping="10" friction="10" />
+			<limit effort="100" velocity="${M_PI / 2.0}" lower="-${joint_3_limit}" upper="${joint_3_limit}"/>
 		</joint>
 		<link name="${name}_link_3">
@@ -133,15 +125,15 @@
 			</inertial>
 			<visual>
-				<origin xyz="0.000 0.028 0.079" rpy="0 0 0" />
-				<geometry>
-					<mesh filename="package://talos_description/meshes/talos_arm/arm3.dae" />
-				</geometry>
-				<material name="Orange" />
+				<origin xyz="0 0 0" rpy="0 0 0" />
+				<geometry>
+					<mesh filename="package://talos_description/meshes/talos_arm/wrist_1_link.stl" />
+				</geometry>
+				<!--material name="Orange" /-->
 			</visual>
 			<collision>
 				<!--<origin xyz="0.000 0.025 0.067" rpy="0 0 0" />-->
-				<origin xyz="0.000 0.028 0.079" rpy="0 0 0" />
-				<geometry>
-					<mesh filename="package://talos_description/meshes/talos_arm/arm3_convex.dae" />
+				<origin xyz="0 0 0" rpy="0 0 0" />
+				<geometry>
+					<mesh filename="package://talos_description/meshes/talos_arm/wrist_1_link.stl" />
 					<!--<box size="0.064 0.054 0.192"/>-->
 				</geometry>
@@ -150,12 +142,11 @@
 		<!-- joint between arm_3_link and arm_4_link -->
 		<joint name="${name}_joint_4" type="revolute">
-			<origin xyz="0.000 0.000 0.135" rpy="0 ${-102.5 * M_PI / 180} 0" />
+			<origin xyz="0 0 0.0715" rpy="0 0 0" />
 			<parent link="${name}_link_3"/>
 			<child link="${name}_link_4"/>
-			<axis xyz="0 1 0" />
+			<axis xyz="0 0 1" />
 			<!--<calibration rising="${arm_4_ref}" falling="${arm_4_ref}"/>-->
-			<dynamics damping="1" friction="1" />
-			<limit effort="${2}" velocity="${M_PI / 2.0}" lower="0" upper="${joint_4_limit}"/>
-			<safety_controller k_position="20" k_velocity="100" soft_lower_limit="0" soft_upper_limit="${joint_4_limit_soft}" />
+			<dynamics damping="10" friction="10" />
+			<limit effort="100" velocity="${M_PI / 2.0}" lower="-${joint_4_limit}" upper="${joint_4_limit}"/>
 		</joint>
 		<link name="${name}_link_4">
@@ -165,15 +156,15 @@
 			</inertial>
 			<visual>
-				<origin xyz="0 -0.010 0.029" rpy="0 0 0"/>
-				<geometry>
-					<mesh filename="package://talos_description/meshes/talos_arm/arm4.dae" />
-				</geometry>
-				<material name="Orange" />
+				<origin xyz="0 0 0.043" rpy="0 0 0"/>
+				<geometry>
+					<mesh filename="package://talos_description/meshes/talos_arm/wrist_2_link.stl" />
+				</geometry>
+				<!--material name="Orange" /-->
 			</visual>
 			<collision>
 				<!--<origin xyz="0 0 0.026" rpy="0 0 0" />-->
-				<origin xyz="0 -0.010 0.029" rpy="0 0 0"/>
-				<geometry>
-					<mesh filename="package://talos_description/meshes/talos_arm/arm4_convex.dae" />
+				<origin xyz="0 0 0.043" rpy="0 0 0"/>
+				<geometry>
+					<mesh filename="package://talos_description/meshes/talos_arm/wrist_2_link.stl" />
 					<!--<box size="0.058 0.100 0.118"/>-->
 				</geometry>
@@ -181,30 +172,90 @@
 		</link>
 		<!-- joint between arm_4_link and arm_5_link -->
-		<joint name="${name}_joint_5" type="revolute">
-			<origin xyz="-0.002 0 0.130" rpy="0 0 ${167.5 * M_PI / 180}" />
+		<joint name="${name}_joint_5" type="fixed">
+			<origin xyz="0 0 0.043" rpy="0 0 0" />
 			<parent link="${name}_link_4"/>
 			<child link="${name}_link_5"/>
-			<axis xyz="0 0 -1" />
+			<axis xyz="0 0 1" />
+			<!--<calibration rising="${arm_4_ref}" falling="${arm_4_ref}"/>-->
+			<dynamics damping="10" friction="10" />
+			<limit effort="100" velocity="${M_PI / 2.0}" lower="-${joint_5_limit}" upper="${joint_5_limit}"/>
+		</joint>
+		<link name="${name}_link_5">
+			<inertial>
+				<mass value="${link_5_mass}"/>
+				<xacro:link_4_inertia_tensor />
+			</inertial>
+			<visual>
+				<origin xyz="0 0 0" rpy="0 0 1.57"/>
+				<geometry>
+					<mesh filename="package://talos_description/meshes/talos_arm/gripper_rail_link.stl" />
+				</geometry>
+				<!--material name="Orange" /-->
+			</visual>
+			<collision>
+				<!--<origin xyz="0 0 0.026" rpy="0 0 0" />-->
+				<origin xyz="0 0 0" rpy="0 0 1.57"/>
+				<geometry>
+					<mesh filename="package://talos_description/meshes/talos_arm/gripper_rail_link.stl" />
+					<!--<box size="0.058 0.100 0.118"/>-->
+				</geometry>
+			</collision>
+		</link>
+		<!-- joint between arm_5_link and arm_6_link -->
+		<joint name="${name}_joint_6" type="prismatic">
+			<origin xyz="0 0 0" rpy="0 0 0" />
+			<parent link="${name}_link_5"/>
+			<child link="${name}_link_6"/>
+			<axis xyz="0 -1 0" />
 			<!--<calibration rising="${arm_5_ref}" falling="${arm_5_ref}"/>-->
-			<dynamics damping="1" friction="1" />
-			<limit effort="1" velocity="${M_PI / 2.0}" lower="0" upper="${joint_5_limit}" />
-                        <safety_controller k_position="20" k_velocity="100" soft_lower_limit="0" soft_upper_limit="${joint_5_limit_soft}" />
-		</joint>
-		<link name="${name}_link_5">
-			<inertial>
-				<mass value="${link_5_mass}"/>
-				<xacro:link_5_inertia_tensor />
-			</inertial>
-			<visual>
-				<origin xyz="0.003 0 -0.034" rpy="0 0 0" />
-				<geometry>
-					<mesh filename="package://talos_description/meshes/talos_arm/arm5.dae" />
-				</geometry>
-				<material name="DarkGrey" />
-			</visual>
-			<collision>
-				<origin xyz="0.003 0 -0.034" rpy="0 0 0" />
-				<geometry>
-					<mesh filename="package://talos_description/meshes/talos_arm/arm5_convex.dae" />
+			<dynamics damping="10" friction="10" />
+			<limit effort="100" velocity="${M_PI / 2.0}" lower="0" upper="${joint_6_limit}" />
+		</joint>
+		<link name="${name}_link_6">
+			<inertial>
+				<mass value="${link_6_mass}"/>
+				<xacro:link_6_inertia_tensor />
+			</inertial>
+			<visual>
+				<origin xyz="0 0 0" rpy="0 0 1.57" />
+				<geometry>
+					<mesh filename="package://talos_description/meshes/talos_arm/gripper_hand_fixed_link.stl" />
+				</geometry>
+				<!--material name="DarkGrey" /-->
+			</visual>
+			<collision>
+				<origin xyz="0 0 0" rpy="0 0 1.57" />
+				<geometry>
+					<mesh filename="package://talos_description/meshes/talos_arm/gripper_hand_fixed_link.stl" />
+					<!--<box size="0.054 0.096 0.030"/>-->
+				</geometry>
+			</collision>
+		</link>
+		<!-- joint between arm_5_link and arm_7_link -->
+		<joint name="${name}_joint_7" type="prismatic">
+			<origin xyz="0 0 0" rpy="0 0 0" />
+			<parent link="${name}_link_5"/>
+			<child link="${name}_link_7"/>
+			<axis xyz="0 1 0" />
+			<!--<calibration rising="${arm_5_ref}" falling="${arm_5_ref}"/>-->
+			<dynamics damping="10" friction="10" />
+			<limit effort="100" velocity="${M_PI / 2.0}" lower="0" upper="${joint_7_limit}" />
+		</joint>
+		<link name="${name}_link_7">
+			<inertial>
+				<mass value="${link_7_mass}"/>
+				<xacro:link_7_inertia_tensor />
+			</inertial>
+			<visual>
+				<origin xyz="0 0 0" rpy="0 0 -1.57" />
+				<geometry>
+					<mesh filename="package://talos_description/meshes/talos_arm/gripper_hand_fixed_link.stl" />
+				</geometry>
+				<!--material name="DarkGrey" /-->
+			</visual>
+			<collision>
+				<origin xyz="0 0 0" rpy="0 0 -1.57" />
+				<geometry>
+					<mesh filename="package://talos_description/meshes/talos_arm/gripper_hand_fixed_link.stl" />
 					<!--<box size="0.054 0.096 0.030"/>-->
 				</geometry>

File: talos_description/urdf/talos_base/base.urdf.xacro (robot description, xacro)
@@ -177,9 +177,9 @@
     </link>
     <!-- base laser front left-->
-    <xacro:sick_tim561_laser name="${name}_laser_left" parent="${name}" ros_topic="scan_left" update_rate="15" min_angle="-2.2" max_angle="2.5" >
+    <xacro:sick_tim561_laser name="${name}_laser_left" parent="${name}" ros_topic="scan_L" update_rate="15" min_angle="-2.2" max_angle="2.5" >
       <origin xyz="0.153 0.279 0.03" rpy="0 0 1.0821" />
     </xacro:sick_tim561_laser>
     <!-- base laser front right-->
-    <xacro:sick_tim561_laser name="${name}_laser_right" parent="${name}" ros_topic="scan_right" update_rate="15" min_angle="-2.5" max_angle="2.2" >
+    <xacro:sick_tim561_laser name="${name}_laser_right" parent="${name}" ros_topic="scan_R" update_rate="15" min_angle="-2.5" max_angle="2.2" >
       <origin xyz="0.153 -0.27 0.03" rpy="0 0 -1.0821" />
     </xacro:sick_tim561_laser>
