Commit message: removed base_footprint

File: talos_description/urdf/talos_base/base.urdf.xacro (robot description, xacro)
@@ -23,10 +23,4 @@
   <xacro:property name="wheel_joint_safety_k_velocity" value="10.0" />
   <xacro:macro name = "talos_base" params="name">
-    <link name="${name}_footprint"/>
-    <joint name="${name}_footprint_joint" type="fixed">
-      <origin xyz="0 0 0" rpy="0 0 0" />
-      <child link="${name}_link" />
-      <parent link="${name}_footprint"/>
-    </joint>
     <link name="${name}_link">
       <inertial>
