Commit message: added imu and realrealsense2 dependecies

File: talos_description/urdf/talos_base/base.gazebo.xacro (robot description, xacro)
@@ -61,3 +61,23 @@
       <minDepth>0.0</minDepth>
     </gazebo>
+    <gazebo reference="imu_link">
+      <gravity>true</gravity>
+      <sensor name="imu_sensor" type="imu">
+        <always_on>true</always_on>
+        <update_rate>100</update_rate>
+        <visualize>true</visualize>
+        <topic>__default_topic__</topic>
+        <plugin filename="libgazebo_ros_imu_sensor.so" name="imu_plugin">
+          <topicName>imu</topicName>
+          <bodyName>imu_link</bodyName>
+          <updateRateHZ>10.0</updateRateHZ>
+          <gaussianNoise>0.0</gaussianNoise>
+          <xyzOffset>0 0 0</xyzOffset>
+          <rpyOffset>0 0 0</rpyOffset>
+          <frameName>imu_link</frameName>
+          <initialOrientationAsReference>false</initialOrientationAsReference>
+        </plugin>
+        <pose>0 0 0 0 0 0</pose>
+      </sensor>
+    </gazebo>
 </robot>

File: talos_description/urdf/talos_base/base.urdf.xacro (robot description, xacro)
@@ -44,4 +44,12 @@
       </collision>
     </link>
+    <link name="imu_link"/>
+    <!-- imu-fixed -->
+    <joint name="fixed_imu" type="fixed">
+      <origin xyz="0.118 0.0 0.05" rpy="0 0 0" />
+      <axis xyz="0 0 1" />
+      <parent link="${name}_link"/>
+      <child link="imu_link" />
+    </joint>
     <!-- front left omni-wheel -->
     <joint name="caster_joint_fl" type="fixed">
