Commit message: added moveit_config

File: talos_description/urdf/materials.urdf.xacro (robot description, xacro)
@@ -1,24 +1,43 @@
 <?xml version="1.0"?>
-<robot>
-  <material name="Orange">
-    <color rgba="1.0 0.4 0.0 1.0"/>
-  </material>
-  <material name="Grey">
-    <color rgba="0.7 0.7 0.7 1.0"/>
-  </material>
-  <material name="DarkGrey">
-    <color rgba="0.3 0.3 0.3 1.0"/>
-  </material>
-  <material name="White">
-    <color rgba="1.0 1.0 1.0 1.0"/>
-  </material>
-  <material name="Black">
-    <color rgba="0.0 0.0 0.0 1.0"/>
-  </material>
-  <material name="Red">
-    <color rgba="1.0 0.0 0.0 1.0"/>
-  </material>
-  <material name="Green">
-    <color rgba="0.0 1.0 0.0 1.0"/>
-  </material>
+<robot xmlns:xacro="http://ros.org/wiki/xacro">
+	<xacro:macro name="material_Orange">
+		<material name="">
+			<color rgba="1.0 0.4 0.0 1.0"/>
+		</material>
+	</xacro:macro>
+	<xacro:macro name="material_Grey">
+		<material name="">
+			<color rgba="0.7 0.7 0.7 1.0"/>
+		</material>
+	</xacro:macro>
+	<xacro:macro name="material_DarkGrey">
+		<material name="">
+			<color rgba="0.3 0.3 0.3 1.0"/>
+		</material>
+	</xacro:macro>
+	<xacro:macro name="material_White">
+		<material name="">
+			<color rgba="1.0 1.0 1.0 1.0"/>
+		</material>
+	</xacro:macro>
+	<xacro:macro name="material_Black">
+		<material name="">
+			<color rgba="0.0 0.0 0.0 1.0"/>
+		</material>
+	</xacro:macro>
+	<xacro:macro name="material_Red">
+		<material name="">
+			<color rgba="1.0 0.0 0.0 1.0"/>
+		</material>
+	</xacro:macro>
+	<xacro:macro name="material_Green">
+		<material name="">
+			<color rgba="0.0 1.0 0.0 1.0"/>
+		</material>
+	</xacro:macro>
+	<xacro:macro name="material_Blue">
+		<material name="">
+			<color rgba="0.0 0.0 1.0 1.0"/>
+		</material>
+	</xacro:macro>
 </robot>

File: talos_description/urdf/robots/talos.urdf.xacro (robot description, xacro)
@@ -15,5 +15,5 @@
   <!--include filename="$(find talos_description)/gazebo/gazebo.urdf.xacro" /-->
   <!-- materials for visualization -->
-  <include filename="$(find talos_description)/urdf/materials.urdf.xacro" />
+  <xacro:include filename="$(find talos_description)/urdf/materials.urdf.xacro" />
   <!-- Now we can start using the macros included above to define the actual talos -->
   <!-- The first use of a macro.  This one was defined in base.urdf.xacro above.
@@ -27,5 +27,5 @@
   <xacro:talos_base name ="base"/>
   <xacro:talos_arm name="arm" parent="base_link">
-    <origin xyz="0.143 0 0.147" rpy="0 0 0" />
+    <origin xyz="0.148 0.0025 0.147" rpy="0 0 0" />
   </xacro:talos_arm>
 </robot>

File: talos_description/urdf/sensors/sick_tim561_laser.urdf.xacro (robot description, xacro)
@@ -20,4 +20,5 @@
         <mesh filename="package://talos_description/meshes/sensors/sick_tim561.stl" />
       </geometry>
+      <xacro:material_Blue />
     </visual>
     <collision>

File: talos_description/urdf/talos_arm/arm.gazebo.xacro (robot description, xacro)
@@ -73,25 +73,28 @@
 		</gazebo>
 		<gazebo reference="${name}_link_6">
-			<!--<material value="youbot/DarkGrey" />-->
-			<turnGravityOff>false</turnGravityOff>
-            <dampingFactor>100000</dampingFactor>
-            <kp>100000.0</kp>
-            <kd>1000.0</kd>
-            <mu1>1.5</mu1>
-            <mu2>1.5</mu2>
-            <fdir>1 0 0</fdir>
-            <maxVel>1.0</maxVel>
+            <mu1>10.5</mu1>
+            <mu2>10.5</mu2>
 		</gazebo>
 		<gazebo reference="${name}_link_7">
-			<!--<material value="youbot/DarkGrey" />-->
-			<turnGravityOff>false</turnGravityOff>
-            <dampingFactor>100000</dampingFactor>
-            <kp>100000.0</kp>
-            <kd>1000.0</kd>
-            <mu1>1.5</mu1>
-            <mu2>1.5</mu2>
-            <fdir>1 0 0</fdir>
-            <maxVel>1.0</maxVel>
+            <mu1>10.5</mu1>
+            <mu2>10.5</mu2>
 		</gazebo>
+        <gazebo>
+        <plugin name="gazebo_grasp_fix" filename="libgazebo_grasp_fix.so">
+                <arm>
+                <arm_name>talos</arm_name>
+                <palm_link>${name}_link_5</palm_link>
+                <gripper_link>${name}_link_6</gripper_link>
+                <gripper_link>${name}_link_7</gripper_link>
+                </arm>
+            <forces_angle_tolerance>100</forces_angle_tolerance>
+            <update_rate>4</update_rate>
+            <grip_count_threshold>4</grip_count_threshold>
+            <max_grip_count>8</max_grip_count>
+            <release_tolerance>0.007</release_tolerance>
+            <disable_collisions_on_attach>false</disable_collisions_on_attach>
+            <contact_topic>__default_topic__</contact_topic>
+            </plugin>
+        </gazebo>
 	</xacro:macro>
 </robot>

File: talos_description/urdf/talos_arm/arm.transmission.xacro (robot description, xacro)
@@ -7,38 +7,73 @@
 	<!-- reduction ratio must not to be 0-->
 	<xacro:macro name="talos_arm_transmission" params="name">
-		<transmission name="${name}_trans_1" type="hardware_interface/EffortJointInterface">
-			<actuator name="${name}_motor_1"/>
-			<joint name="${name}_joint_1"/>
-			<mechanicalReduction>1</mechanicalReduction>
+		<transmission name="${name}_trans_0">
+			<type>transmission_interface/SimpleTransmission</type>
+			<joint name="${name}_joint_0">
+				<hardwareInterface>hardware_interface/EffortJointInterface</hardwareInterface>
+			</joint>
+			<actuator name="${name}_joint_0_actr">
+				<hardwareInterface>hardware_interface/EffortJointInterface</hardwareInterface>
+				<mechanicalReduction>1</mechanicalReduction>
+			</actuator>
 		</transmission>
-		<transmission name="${name}_trans_2" type="hardware_interface/EffortJointInterface">
-			<actuator name="${name}_motor_2"/>
-			<joint name="${name}_joint_2"/>
-			<mechanicalReduction>1</mechanicalReduction>
+		<transmission name="${name}_trans_1">
+			<type>transmission_interface/SimpleTransmission</type>
+			<joint name="${name}_joint_1">
+				<hardwareInterface>hardware_interface/EffortJointInterface</hardwareInterface>
+			</joint>
+			<actuator name="${name}_joint_1_actr">
+				<hardwareInterface>hardware_interface/EffortJointInterface</hardwareInterface>
+				<mechanicalReduction>1</mechanicalReduction>
+			</actuator>
 		</transmission>
-		<transmission name="${name}_trans_3" type="hardware_interface/EffortJointInterface">
-			<actuator name="${name}_motor_3"/>
-			<joint name="${name}_joint_3"/>
-			<mechanicalReduction>1</mechanicalReduction>
+		<transmission name="${name}_trans_2">
+			<type>transmission_interface/SimpleTransmission</type>
+			<joint name="${name}_joint_2">
+				<hardwareInterface>hardware_interface/EffortJointInterface</hardwareInterface>
+			</joint>
+			<actuator name="${name}_joint_2_actr">
+				<hardwareInterface>hardware_interface/EffortJointInterface</hardwareInterface>
+				<mechanicalReduction>1</mechanicalReduction>
+			</actuator>
 		</transmission>
-		<transmission name="${name}_trans_4" type="hardware_interface/EffortJointInterface">
-			<actuator name="${name}_motor_4"/>
-			<joint name="${name}_joint_4"/>
-			<mechanicalReduction>1</mechanicalReduction>
+		<transmission name="${name}_trans_3">
+			<type>transmission_interface/SimpleTransmission</type>
+			<joint name="${name}_joint_3">
+				<hardwareInterface>hardware_interface/EffortJointInterface</hardwareInterface>
+			</joint>
+			<actuator name="${name}_joint_3_actr">
+				<hardwareInterface>hardware_interface/EffortJointInterface</hardwareInterface>
+				<mechanicalReduction>1</mechanicalReduction>
+			</actuator>
 		</transmission>
-		<transmission name="${name}_trans_5" type="hardware_interface/EffortJointInterface">
-			<actuator name="${name}_motor_5"/>
-			<joint name="${name}_joint_5"/>
-			<mechanicalReduction>1</mechanicalReduction>
+		<transmission name="${name}_trans_4">
+			<type>transmission_interface/SimpleTransmission</type>
+			<joint name="${name}_joint_4">
+				<hardwareInterface>hardware_interface/EffortJointInterface</hardwareInterface>
+			</joint>
+			<actuator name="${name}_joint_4_actr">
+				<hardwareInterface>hardware_interface/EffortJointInterface</hardwareInterface>
+				<mechanicalReduction>1</mechanicalReduction>
+			</actuator>
 		</transmission>
-		<transmission name="${name}_trans_6" type="hardware_interface/EffortJointInterface">
-			<actuator name="${name}_motor_6"/>
-			<joint name="${name}_joint_6"/>
-			<mechanicalReduction>1</mechanicalReduction>
+		<transmission name="${name}_trans_6">
+			<type>transmission_interface/SimpleTransmission</type>
+			<joint name="${name}_joint_6">
+				<hardwareInterface>hardware_interface/EffortJointInterface</hardwareInterface>
+			</joint>
+			<actuator name="${name}_joint_6_actr">
+				<hardwareInterface>hardware_interface/EffortJointInterface</hardwareInterface>
+				<mechanicalReduction>1</mechanicalReduction>
+			</actuator>
 		</transmission>
-		<transmission name="${name}_trans_7" type="hardware_interface/EffortJointInterface">
-			<actuator name="${name}_motor_7"/>
-			<joint name="${name}_joint_7"/>
-			<mechanicalReduction>1</mechanicalReduction>
+		<transmission name="${name}_trans_7">
+			<type>transmission_interface/SimpleTransmission</type>
+			<joint name="${name}_joint_7">
+				<hardwareInterface>hardware_interface/EffortJointInterface</hardwareInterface>
+			</joint>
+			<actuator name="${name}_joint_7_actr">
+				<hardwareInterface>hardware_interface/EffortJointInterface</hardwareInterface>
+				<mechanicalReduction>1</mechanicalReduction>
+			</actuator>
 		</transmission>
 	</xacro:macro>

File: talos_description/urdf/talos_arm/arm.urdf.xacro (robot description, xacro)
@@ -13,8 +13,11 @@
 		</xacro:sensor_d435>
 		<!-- joint between base_link and arm_0_link -->
-		<joint name="${name}_joint_0" type="fixed" >
+		<joint name="${name}_joint_0" type="revolute" >
 			<xacro:insert_block name="origin" />
 			<parent link="${parent}" />
 			<child link="${name}_link_0" />
+			<axis xyz="0 0 1"/>
+			<dynamics damping="10" friction="5" />
+			<limit effort="100" velocity="${M_PI / 2.0}" lower="-${joint_0_limit}" upper="${joint_0_limit}"/>
 		</joint>
 		<link name="${name}_link_0">
@@ -30,5 +33,5 @@
 					<mesh filename="package://talos_description/meshes/talos_arm/shoulder_link.stl" />
 				</geometry>
-				<!--material name="DarkGrey" /-->
+				<xacro:material_Black />
 			</visual>
 			<collision>
@@ -48,5 +51,5 @@
 			<axis xyz="0 1 0"/>
 			<!--<calibration rising="${arm_1_ref}" falling="${arm_1_ref}"/>-->
-			<dynamics damping="10" friction="10" />
+			<dynamics damping="10" friction="5" />
 			<!-- damping - N*s/m, N*s*m/rad -->
 			<!-- friction - N, N*m -->
@@ -68,5 +71,5 @@
 					<mesh filename="package://talos_description/meshes/talos_arm/biceps_link.stl" />
 				</geometry>
-				<!--<material name="Orange" />-->
+				<xacro:material_Black />
 			</visual>
 			<collision>
@@ -86,5 +89,5 @@
 			<axis xyz="0 1 0"/>
 			<!--<calibration rising="${arm_2_ref}" falling="${arm_2_ref}"/>-->
-			<dynamics damping="10" friction="10" />
+			<dynamics damping="10" friction="5" />
 			<limit effort="100" velocity="${M_PI / 2.0}" lower="-${joint_2_limit}" upper="${joint_2_limit}"/>
 		</joint>
@@ -99,5 +102,5 @@
 					<mesh filename="package://talos_description/meshes/talos_arm/forearm_link.stl" />
 				</geometry>
-				<!--material name="Black" /-->
+				<xacro:material_Black />
 			</visual>
 			<collision>
@@ -116,5 +119,5 @@
 			<child link="${name}_link_3"/>
 			<axis xyz="0 1 0"/>
-			<dynamics damping="10" friction="10" />
+			<dynamics damping="10" friction="5" />
 			<limit effort="100" velocity="${M_PI / 2.0}" lower="-${joint_3_limit}" upper="${joint_3_limit}"/>
 		</joint>
@@ -129,5 +132,5 @@
 					<mesh filename="package://talos_description/meshes/talos_arm/wrist_1_link.stl" />
 				</geometry>
-				<!--material name="Orange" /-->
+				<xacro:material_Black />
 			</visual>
 			<collision>
@@ -147,5 +150,5 @@
 			<axis xyz="0 0 1" />
 			<!--<calibration rising="${arm_4_ref}" falling="${arm_4_ref}"/>-->
-			<dynamics damping="10" friction="10" />
+			<dynamics damping="10" friction="5" />
 			<limit effort="100" velocity="${M_PI / 2.0}" lower="-${joint_4_limit}" upper="${joint_4_limit}"/>
 		</joint>
@@ -160,5 +163,5 @@
 					<mesh filename="package://talos_description/meshes/talos_arm/wrist_2_link.stl" />
 				</geometry>
-				<!--material name="Orange" /-->
+				<xacro:material_Black />
 			</visual>
 			<collision>
@@ -178,5 +181,5 @@
 			<axis xyz="0 0 1" />
 			<!--<calibration rising="${arm_4_ref}" falling="${arm_4_ref}"/>-->
-			<dynamics damping="10" friction="10" />
+			<dynamics damping="10" friction="5" />
 			<limit effort="100" velocity="${M_PI / 2.0}" lower="-${joint_5_limit}" upper="${joint_5_limit}"/>
 		</joint>
@@ -191,5 +194,5 @@
 					<mesh filename="package://talos_description/meshes/talos_arm/gripper_rail_link.stl" />
 				</geometry>
-				<!--material name="Orange" /-->
+				<xacro:material_Black />
 			</visual>
 			<collision>
@@ -209,6 +212,6 @@
 			<axis xyz="0 -1 0" />
 			<!--<calibration rising="${arm_5_ref}" falling="${arm_5_ref}"/>-->
-			<dynamics damping="10" friction="10" />
-			<limit effort="100" velocity="${M_PI / 2.0}" lower="0" upper="${joint_6_limit}" />
+			<dynamics damping="1000"/>
+			<limit effort="10000" velocity="0.5" lower="0" upper="${joint_6_limit}" />
 		</joint>
 		<link name="${name}_link_6">
@@ -222,5 +225,5 @@
 					<mesh filename="package://talos_description/meshes/talos_arm/gripper_hand_fixed_link.stl" />
 				</geometry>
-				<!--material name="DarkGrey" /-->
+				<xacro:material_Black />
 			</visual>
 			<collision>
@@ -238,7 +241,7 @@
 			<child link="${name}_link_7"/>
 			<axis xyz="0 1 0" />
+			<dynamics damping="1000"/>
 			<!--<calibration rising="${arm_5_ref}" falling="${arm_5_ref}"/>-->
-			<dynamics damping="10" friction="10" />
-			<limit effort="100" velocity="${M_PI / 2.0}" lower="0" upper="${joint_7_limit}" />
+			<limit effort="10000" velocity="0.5" lower="0" upper="${joint_7_limit}" />
 		</joint>
 		<link name="${name}_link_7">
@@ -252,5 +255,5 @@
 					<mesh filename="package://talos_description/meshes/talos_arm/gripper_hand_fixed_link.stl" />
 				</geometry>
-				<!--material name="DarkGrey" /-->
+				<xacro:material_Black />
 			</visual>
 			<collision>

File: talos_description/urdf/talos_arm/limits.urdf.xacro (robot description, xacro)
@@ -4,5 +4,6 @@
 	<xacro:property name="M_PI" value="3.1415926535897931" />
     <xacro:property name="threshold" value="0.01" />
-	<!-- arm limits positions (deg) -->
+	<!-- arm limits positions (rad) -->
+	<xacro:property name="joint_0_limit" value="3.1415" />
 	<xacro:property name="joint_1_limit" value="3.1415" />
 	<xacro:property name="joint_2_limit" value="1.571" />
@@ -58,9 +59,9 @@
 	<xacro:macro name="link_6_inertia_tensor">
 		<origin xyz="0 0 0" rpy="0 0 1.57" />
-		<inertia ixx="0.000280" ixy="0.000000" ixz="0.000000" iyy="0.000339" iyz="0.000000" izz="0.000119" />
+		<inertia ixx="0.01" ixy="0.000000" ixz="0.000000" iyy="0.01" iyz="0.000000" izz="0.01" />
 	</xacro:macro>
 	<xacro:macro name="link_7_inertia_tensor">
 		<origin xyz="0 0 0" rpy="0 0 -1.57" />
-		<inertia ixx="0.000280" ixy="0.000000" ixz="0.000000" iyy="0.000339" iyz="0.000000" izz="0.000119" />
+		<inertia ixx="0.01" ixy="0.000000" ixz="0.000000" iyy="0.01" iyz="0.000000" izz="0.01" />
 	</xacro:macro>
 </robot>

File: talos_description/urdf/talos_base/base.gazebo.xacro (robot description, xacro)
@@ -5,4 +5,9 @@
         xmlns:xacro="http://ros.org/wiki/xacro">
   <xacro:macro name="talos_base_gazebo">
+    <gazebo>
+        <plugin name="gazebo_ros_control" filename="libgazebo_ros_control.so">
+            <robotNamespace>/talos</robotNamespace>
+        </plugin>
+    </gazebo>
     <gazebo>
       <plugin name="object_controller" filename="libgazebo_ros_planar_move.so">
@@ -56,5 +61,3 @@
       <minDepth>0.0</minDepth>
     </gazebo>
-    <gazebo reference="caster_link_b">
-    </gazebo>
 </robot>

File: talos_description/urdf/talos_base/base.transmission.xacro (robot description, xacro)
@@ -11,7 +11,9 @@
     <transmission name="wheel_trans_fl">
       <type>transmission_interface/SimpleTransmission</type>
-      <joint name="wheel_joint_fl"/>
+      <joint name="wheel_joint_fl">
+				<hardwareInterface>hardware_interface/VelocityJointInterface</hardwareInterface>
+			</joint>
       <actuator name="wheel_motor_fl">
-        <hardwareInterface>VelocityJointInterface</hardwareInterface>
+        <hardwareInterface>hardware_interface/VelocityJointInterface</hardwareInterface>
         <mechanicalReduction>${wheel_mechanical_reduction}</mechanicalReduction>
       </actuator>
@@ -20,7 +22,9 @@
     <transmission name="wheel_trans_fr">
       <type>transmission_interface/SimpleTransmission</type>
-      <joint name="wheel_joint_fr"/>
+      <joint name="wheel_joint_fr">
+				<hardwareInterface>hardware_interface/VelocityJointInterface</hardwareInterface>
+			</joint>
       <actuator name="wheel_motor_fr">
-        <hardwareInterface>VelocityJointInterface</hardwareInterface>
+        <hardwareInterface>hardware_interface/VelocityJointInterface</hardwareInterface>
         <mechanicalReduction>${wheel_mechanical_reduction}</mechanicalReduction>
       </actuator>
@@ -29,7 +33,9 @@
     <transmission name="wheel_trans_b">
       <type>transmission_interface/SimpleTransmission</type>
-      <joint name="wheel_joint_b"/>
+      <joint name="wheel_joint_b">
+				<hardwareInterface>hardware_interface/VelocityJointInterface</hardwareInterface>
+			</joint>
       <actuator name="wheel_motor_b">
-        <hardwareInterface>VelocityJointInterface</hardwareInterface>
+        <hardwareInterface>hardware_interface/VelocityJointInterface</hardwareInterface>
         <mechanicalReduction>${wheel_mechanical_reduction}</mechanicalReduction>
       </actuator>

File: talos_description/urdf/talos_base/base.urdf.xacro (robot description, xacro)
@@ -34,4 +34,5 @@
           <mesh filename="package://talos_description/meshes/talos_base/talos_base.stl"/>
         </geometry>
+        <xacro:material_DarkGrey />
       </visual>
       <collision>
@@ -77,4 +78,5 @@
           <mesh filename="package://talos_description/meshes/talos_base/omniwheel.stl" />
         </geometry>
+        <xacro:material_DarkGrey />
       </visual>
       <collision>
@@ -119,4 +121,5 @@
           <mesh filename="package://talos_description/meshes/talos_base/omniwheel.stl" />
         </geometry>
+        <xacro:material_DarkGrey />
       </visual>
       <collision>
@@ -162,4 +165,5 @@
           <mesh filename="package://talos_description/meshes/talos_base/omniwheel.stl" />
         </geometry>
+        <xacro:material_DarkGrey />
       </visual>
       <collision>
