Commit message: fixed arm_urdf issues

File: talos_description/urdf/talos_arm/arm.urdf.xacro (robot description, xacro)
@@ -103,4 +103,5 @@
 				</geometry>
 				<xacro:material_Black />
+			</visual>
 			<collision>
 				<!--<origin xyz="0.001 -0.041 0.074" rpy="0 0 0" />-->
@@ -183,8 +184,8 @@
 			<limit effort="100" velocity="${M_PI / 2.0}" lower="-${joint_5_limit}" upper="${joint_5_limit}"/>
 		</joint>
-		<link name="${name}_link_6">
+		<link name="${name}_link_5">
 			<inertial>
 				<mass value="${link_5_mass}"/>
-				<xacro:link_4_inertia_tensor />
+				<xacro:link_5_inertia_tensor />
 			</inertial>
 			<visual>
