Commit message: additional objects

File: talos_description/urdf/talos_arm/arm.gazebo.xacro (robot description, xacro)
@@ -62,6 +62,4 @@
 		</gazebo>
 		<gazebo reference="${name}_link_5">
-			<!--<material value="youbot/DarkGrey" />-->
-			<turnGravityOff>false</turnGravityOff>
             <dampingFactor>100000</dampingFactor>
             <kp>100000.0</kp>
@@ -82,10 +80,10 @@
         <gazebo>
         <plugin name="gazebo_grasp_fix" filename="libgazebo_grasp_fix.so">
-                <arm>
-                <arm_name>talos</arm_name>
-                <palm_link>${name}_link_5</palm_link>
-                <gripper_link>${name}_link_6</gripper_link>
-                <gripper_link>${name}_link_7</gripper_link>
-                </arm>
+                  <arm>
+                  <arm_name>talos</arm_name>
+                  <palm_link>${name}_link_ee</palm_link>
+                  <gripper_link>${name}_link_6</gripper_link>
+                  <gripper_link>${name}_link_7</gripper_link>
+                  </arm>
             <forces_angle_tolerance>100</forces_angle_tolerance>
             <update_rate>4</update_rate>

File: talos_description/urdf/talos_arm/arm.urdf.xacro (robot description, xacro)
@@ -265,4 +265,12 @@
 			</collision>
 		</link>
+		<!-- joint between arm_5_link and arm_link_ee -->
+		<joint name="${name}_joint_ee" type="fixed">
+			<origin xyz="0 0 0.05" rpy="0 0 0" />
+			<parent link="${name}_link_5"/>
+			<child link="${name}_link_ee"/>
+			<axis xyz="0 1 0" />
+		</joint>
+		<link name="${name}_link_ee"/>
 		<!-- extensions -->
 		<xacro:talos_arm_gazebo name="${name}" />
